Commit message: add floor

File: src/ur_softhand_description/urdf/my_robot_cell_macro.xacro (robot description, xacro)
@@ -40,4 +40,33 @@
       <origin xyz="0 0 0" rpy="0 0 0"/> <!-- Ajusta el offset según sea necesario -->
     </joint>
+    <!-- Agregar un plano al entorno -->
+    <link name="floor">
+      <visual>
+        <geometry>
+          <box size="2.0 2.0 0.01"/>
+          <!-- Dimensiones del plano 20m x 20m x 0.01m -->
+        </geometry>
+        <origin xyz="0 0 -0.005" rpy="0 0 0"/> <!-- Colocado en z=0 -->
+        <material name="floor_material">
+          <color rgba="0.8 0.8 0.8 1.0"/> <!-- Color gris claro -->
+        </material>
+      </visual>
+      <collision>
+        <geometry>
+          <box size="20.0 20.0 0.01"/>
+        </geometry>
+        <origin xyz="0 0 -0.005" rpy="0 0 0"/>
+      </collision>
+      <inertial>
+        <mass value="1.0"/> <!-- Masa arbitraria -->
+        <origin xyz="0 0 -0.005" rpy="0 0 0"/>
+        <inertia ixx="0.01" iyy="0.01" izz="0.01" ixy="0.0" ixz="0.0" iyz="0.0"/>
+      </inertial>
+    </link>
+    <joint name="floor_to_world" type="fixed">
+      <parent link="world"/>
+      <child link="floor"/>
+      <origin xyz="0 0 0" rpy="0 0 0"/>
+    </joint>
   </xacro:macro>
 </robot>
